File: Pelt_Proj/Hbridges.sch (KiCad schematic (older format))
At the start: 24 parts

Commit message: with new hbridge file
Connections:
- net INH_A_1: now reaches R?.2
- net IS_1: now reaches R?.1, U?.6 (IS), U?.6 (IS)
- net IN_A_1: now reaches R?.2
- net IN_B_1: now reaches R?.2
- net INH_B_1: now reaches R?.2
- net INH_A_2: now reaches R?.2
- net IS_2: now reaches R?.1, U?.6 (IS), U?.6 (IS)
- net IN_A_2: now reaches R?.2
- net IN_B_2: now reaches R?.2
- net INH_B_2: now reaches R?.2
Other:
- note added: "Pelt 1"
- note added: "Pelt 2"
- moved on the sheet: C?, P?, R?, U?

Commit message: Near complet first draft of schematics
Parts:
- removed P? (x2): CONN_01X02, symbol CONN_01X02
- added P5: CONN_01X04, symbol CONN_01X04
- gave numbers to parts that had none: 22
Connections:
- net INH_A_2 is gone; now on net INH: R26.2
- net INH_B_2 is gone; now on net IN_B: R30.2
- net IN_A_2 is gone; now on net IN_A: R25.2
- net IN_B_1 is gone; now on net INH: R21.2
- net IN_B_2 is gone; now on net INH: R28.2
- net at U13.4 (OUT): now also P5.2 (P2)
- net at U12.4 (OUT): now also P5.1 (P1)
- net at U15.4 (OUT): now also P5.4 (P4)
- net at U14.4 (OUT): now also P5.3 (P3)
- net INH_A_1 renamed INH
- net INH_B_1 renamed IN_B
- net IN_A_1 renamed IN_A
