File: Pelt_Proj/Pelt_Proj.sch (KiCad schematic (older format))
At the start: 94 parts, among them P1 CONN_01X02, P2 CONN_01X03

Commit message: with dual therm circuits
Parts:
- removed C2, C?: 470nF, symbol C
- removed C?: 0.1u, symbol C
- removed P1: CONN_01X02, symbol CONN_01X02
- removed P?: CONN_01X10, symbol CONN_01X10
- removed Q? (x6): Q_PNP_BCE, symbol Q_PNP_BCE-RESCUE-Pelt_Proj
- removed Q? (x4): Q_NMOS_DGS, symbol Q_NMOS_DGS-RESCUE-Pelt_Proj
- removed Q? (x2): Q_PMOS_DGS, symbol Q_PMOS_DGS-RESCUE-Pelt_Proj
- removed R1, R11, R12, R2, R3, R4: 1k, symbol R
- removed R10, R7: 3.3k, symbol R
- removed R5, R? (x25): 10k, symbol R
- removed R6, R?: R, symbol R
- removed R? (x4): 5k, symbol R
- removed R? (x2): 250, symbol R
- removed R? (x2): 100k, symbol R
- removed R?: 470, symbol R
- removed RV? (x8): 100, symbol POT
- removed U?: LTC1448, symbol LTC1448
- removed U? (x10): OP275, symbol OP275
- removed U?: TL071, symbol TL071
- removed U? (x2): BTN7906, symbol BTN7906
- added ???: KEYPAD4X4, symbol KEYPAD4X4
- added C?: 0.01u, symbol C
- added R?: 30k, symbol R
- added U? (x2): OP2137, symbol OP2137
Connections:
- net CS1: no longer U?.16 (RF2/AN7/C1OUT)
- net GND: now also C?.2, R?.2, U?.4 (V-), U?.4 (V-)
- net VDD: now also U?.8 (V+), U?.8 (V+)
- net CS2: no longer names the net of U?.15 (RF3/AN8/C2INB/CTMUI)
- net CS3: no longer names the net of U?.14 (RF4/AN9/C2INA)
- net CS4: no longer names the net of U?.13 (RF5/AN10/CVREF/C1INB)
- net CS5: no longer names the net of U?.12 (RF6/AN11/C1INA)
- net CS6: no longer names the net of U?.11 (RF7/AN5/SS1)
- net CS7: no longer names the net of U?.8 (RG4/RTCC/T7CKI(2)/T5G/CCP5/AN16/P1D/C3INC)
- net CS8: no longer names the net of U?.6 (RG3/CCP4/AN17/P3D/C3INB)
- net THERM renamed THERM_1
- net THERM_1: now also U?.3 (+)
- new net THERM_2: C?.1, R?.1, U?.5 (+)
- new net THERM_IN_1: U?.1, U?.2 (-)
- new net THERM_IN_2: U?.6 (-), U?.7
Other:
- note removed: "Current Source 1"
- note removed: "Current Source 2"
- note removed: "Current Source 3"
- note removed: "Current Source 4"
- note removed: "Current Source 5"
- note removed: "Current Source 6"
- note removed: "GND"
- note removed: "Master Therm"
- note removed: "Peltier"
- note removed: "Sensor Conn"
- moved on the sheet: C?, DS?, R9, R?, RV1

Commit message: Near complet first draft of schematics
Parts:
- added P4: CONN_01X16, symbol CONN_01X16
- gave numbers to parts that had none: 11
Connections:
- net THERM_IN is gone; now on net THERM_IN_1: U1.17 (RF1/AN6/C2OUT/CTDIN)
- net GND: now also P4.1 (P1); no longer C2.2, C3.2, R2.2, R3.2, U2.4 (V-), U2.4 (V-)
- net Hbridges/IS_1: now also U1.44 (RB4/KBI0)
- net Hbridges/IS_2: now also U1.43 (RB5/KBI1/T3CKI/T1G)
- net THERM_1: now also P4.15 (P15); no longer C2.1, R2.1, U2.3 (+)
- net THERM_2: now also P4.16 (P16)
- net THERM_IN_1: no longer U2.1, U2.2 (-)
- net THERM_IN_2: now also U1.16 (RF2/AN7/C1OUT)
- net JP1: now reaches U1.1 (RE1/WR/P2C)
- net JP1: now also P4.3 (P3)
- net HCE2: now reaches U1.11 (RF7/AN5/SS1)
- net HCE1: now reaches U1.12 (RF6/AN11/C1INA)
- net JP10: now reaches U1.13 (RF5/AN10/CVREF/C1INB)
- net JP10: now also P4.12 (P12)
- net JP9: now reaches U1.14 (RF4/AN9/C2INA)
- net JP9: now also P4.11 (P11)
- net JP8: now reaches U1.15 (RF3/AN8/C2INB/CTMUI)
- net JP8: now also P4.10 (P10)
- net JP0: now reaches U1.2 (RE0/RD/P2D)
- net JP0: now also P4.2 (P2)
- net at U1.21 (RA3/AN3/VREF+): now also ??1.4 (R4)
- net at U1.22 (RA2/AN2/VREF): now also ??1.3 (R3)
- net at U1.23 (RA1/AN1): now also ??1.2 (R2)
- net at U1.24 (RA0/AN0/ULPWU): now also ??1.1 (R1)
- net at U1.27 (RA5/AN4/T1CKI/T3G/): now also ??1.6 (C2)
- net at U1.28 (RA4/T0CKI): now also ??1.5 (C1)
- net Pelt_Proj_JoeCrt/A1: now reaches U1.29 (RC1/SOSCI/ECCP2/P2A)
- net Pelt_Proj_JoeCrt/A0: now reaches U1.30 (RC0/SOSCO/SCLKI)
- net Pelt_Proj_JoeCrt/A2: now reaches U1.33 (RC2/ECCP1/P1A)
- net SDI: now reaches U1.35 (RC4/SDI1/SDA1)
- net at U1.39 (OSC1/CLKI/RA7): now also ??1.8 (C4)
- net at U1.40 (OSC2/CLKO/RA6): now also ??1.7 (C3)
- net JP7: now reaches U1.59 (RE7/ECCP2/P2A)
- net JP7: now also P4.9 (P9)
- net JP6: now reaches U1.60 (RE6/P1B/CCP6)
- net JP6: now also P4.8 (P8)
- net JP5: now reaches U1.61 (RE5/P1C/CCP7)
- net JP5: now also P4.7 (P7)
- net JP4: now reaches U1.62 (RE4/P3B/CCP8)
- net JP4: now also P4.6 (P6)
- net JP3: now reaches U1.63 (RE3/P3C/CCP9/REFO)
- net JP3: now also P4.5 (P5)
- net JP2: now reaches U1.64 (RE2/CS/P2B/CCP10)
- net JP2: now also P4.4 (P4)
- net microsd/MicroSD_CS: now reaches U1.8 (RG4/RTCC/T7CKI(2)/T5G/CCP5/AN16/P1D/C3INC)
- net CS1 renamed Pelt_Proj_JoeCrt/D2A_CS
- net RB0 renamed Hbridges/INH
- net RB1 renamed Pelt_Proj_JoeCrt/A2D_CS
- net RB2 renamed Hbridges/IN_B
- net RB3 renamed Hbridges/IN_A
- net SCL1 renamed SCLK
- net SDO1 renamed SDO
- new net: C2.1, R2.1, U2.3 (+)
- new net: U2.1, U2.2 (-)
- new net -5V: C2.2, C3.2, R2.2, R3.2, U2.4 (V-), U2.4 (V-)
- new net Sensor_1: P4.13 (P13)
- new net Sensor_2: P4.14 (P14)
- no-connect marks 6 -> 4
Other:
- note added: "LED Register"
- note added: "Test Connector\nJumpers(11)\nThermistors(2)\nSensor Connections(2)\nGND"
- note added: "Thermistor Interfaces"
- moved on the sheet: ??1, C2, C3, DS1, R2, R3, R9, RV1, U2A, U2B
