File: Pelt_Proj/Pelt_Proj_JoeCrt.sch (KiCad schematic (older format))
At the start: 27 parts

Commit message: with dual therm circuits
Parts:
- added C? (x2): 10uF, symbol CP_Small
- added IC?: ICL7660CPA, maxim-10-DIL08, symbol ICL7660CPA
- added P?: CONN_01X02, symbol CONN_01X02
- added Q?: 2N3906, symbol 2N3906
- added Q?: ZVP2110A, symbol ZVP2110A
- added Q?: 2N7000, symbol 2N7000
- added R? (x3): 10k, symbol R
- added R?: RH, symbol R
- added R?: RL, symbol R
- added U?: OP2277, symbol OP2277
Connections:
- net labels added: 12V, High_Current_Enable_1, High_Current_Enable_2
- net labels removed: High_Current_Enable, VOUTb
- wire segments 83 -> 121
Other:
- note added: "-5V reference"
- note added: "5v precision reference"
- note added: "Regulated 10V"
- note added: "Regulated 5V"
- moved on the sheet: ???, C?, D?, IC?, L?, P?, Q?, R?, U?, U?A

Commit message: Near complet first draft of schematics
Parts:
- removed P? (x2): CONN_01X02, symbol CONN_01X02
- U9: renamed from ???; symbol LM2575-RESCUE-Pelt_Proj -> LM2575
- gave numbers to parts that had none: 36
Connections:
- net D2A_Data_Input is gone; now on net SCLK: U7.1 (CLK)
- net +12V: now also U9.P$1 (IN); no longer U9.1 (IN)
- net +5V: now also U9.P$4 (FB); no longer U9.4 (FB)
- net GND: now also U9.P$3 (GND), U9.P$5 (EN); no longer R16.2, U9.3 (GND), U9.5 (EN)
- net at L1.2: now also U9.P$2 (OUT); no longer U9.2 (OUT)
- net Sensor_1: now reaches IC1.4 (S1), Q1.3 (C)
- net Sensor_2: now reaches IC1.5 (S2), Q4.3 (C)
- net at IC1.8 (D): now also U5.2 (-)
- net at U5.1, U6.2 (IN+): now also U5.3 (+)
- net at Q4.2 (B): now also U8.7; no longer U8.1
- net at Q4.1 (E), R13.2: now also U8.6 (-); no longer U8.2 (-)
- net at R10.2, R11.1: now also U8.5 (+); no longer U8.3 (+)
- net 5V_Ref renamed 5V_REF
- net A/DStart renamed A2D_CS
- net Clock renamed SCLK
- net D2A_Clock renamed MOSI
- net D2A_Load: no longer names the net of U7.3 (_CS/LD)
- net DataOut renamed MISO
Other:
- note added: "SPI Connections"
- moved on the sheet: C10, C13, C6, C7, C8, C9, D1, IC2, L1, U5A, U6
