File: Pelt_Proj/Pelt_Proj_PowerReg.sch (KiCad schematic (older format))
At the start: 6 parts

Commit message: with dual therm circuits
Parts:
- removed P?: CONN_01X02, symbol CONN_01X02
Connections:
- net labels added: 12V
- wire segments 16 -> 14
Other:
- note added: "Main Power Connector"
Changed lines of the file:
@@
 LIBS:jfw-pwm1
 LIBS:mylib
+LIBS:maxim-10
+LIBS:keypad4x4_ece
 LIBS:Pelt_Proj-cache
 EELAYER 25 0
 EELAYER END
-$Descr A4 11693 8268
+$Descr USLetter 11000 8500
 encoding utf-8
 Sheet 2 4
@@
 	1    0    0    -1
 $EndComp
-$Comp
-L CONN_01X02 P?
-U 1 1 5568F486
-P 4150 3850
-F 0 "P?" H 4150 4000 50  0000 C CNN
-F 1 "CONN_01X02" V 4250 3850 50  0000 C CNN
-F 2 "" H 4150 3850 60  0000 C CNN
-F 3 "" H 4150 3850 60  0000 C CNN
-	1    4150 3850
-	-1   0    0    1
-$EndComp
 Wire Wire Line
 	5375 4050 5375 4125
@@
 	5950 3750 5950 3700
 Wire Wire Line
-	4350 3750 4975 3750
-Wire Wire Line
 	4800 3750 4800 3700
-Wire Wire Line
-	4350 4050 5375 4050
-Wire Wire Line
-	4350 3750 4350 3800
-Connection ~ 4800 3750
-Wire Wire Line
-	4350 3900 4350 4050
-Connection ~ 4800 4050
 $Comp
 L +12V #PWR?
@@
 Text HLabel 5950 3750 2    60   Input ~ 0
 VDD
+Text GLabel 4475 2875 1    60   Input ~ 12
+12V
+Wire Wire Line
+	4825 4050 5375 4050
+Wire Wire Line
+	4975 3750 4800 3750
+Text Notes 2875 3025 0    60   Italic 12
+Main Power Connector
 $EndSCHEMATC

Commit message: Near complet first draft of schematics
Parts:
- added D?: LED, symbol LED
- added R?: R_Small, symbol R_Small
- gave numbers to parts that had none: 5
Connections:
- wire segments 14 -> 18
Changed lines of the file:
@@
 $Descr USLetter 11000 8500
 encoding utf-8
-Sheet 2 4
+Sheet 2 5
 Title ""
 Date ""
@@
 $EndDescr
 $Comp
-L +12V #PWR?
+L +12V #PWR22
 U 1 1 5568F466
 P 4800 3700
-F 0 "#PWR?" H 4800 3550 50  0001 C CNN
+F 0 "#PWR22" H 4800 3550 50  0001 C CNN
 F 1 "+12V" H 4800 3840 50  0000 C CNN
 F 2 "" H 4800 3700 60  0000 C CNN
@@
 $EndComp
 $Comp
-L GND #PWR?
+L GND #PWR24
 U 1 1 5568F46C
 P 5375 4125
-F 0 "#PWR?" H 5375 3875 50  0001 C CNN
+F 0 "#PWR24" H 5375 3875 50  0001 C CNN
 F 1 "GND" H 5375 3975 50  0000 C CNN
 F 2 "" H 5375 4125 60  0000 C CNN
@@
 $EndComp
 $Comp
-L LM7805CT U?
+L LM7805CT U4
 U 1 1 5568F472
 P 5375 3800
-F 0 "U?" H 5175 4000 40  0000 C CNN
+F 0 "U4" H 5175 4000 40  0000 C CNN
 F 1 "LM7805CT" H 5375 4000 40  0000 L CNN
 F 2 "TO-220" H 5375 3900 30  0000 C CIN
@@
 $EndComp
 $Comp
-L VDD #PWR?
+L VDD #PWR26
 U 1 1 5568F479
 P 5950 3700
-F 0 "#PWR?" H 5950 3550 50  0001 C CNN
+F 0 "#PWR26" H 5950 3550 50  0001 C CNN
 F 1 "VDD" H 5950 3850 50  0000 C CNN
 F 2 "" H 5950 3700 60  0000 C CNN
@@
 $EndComp
 $Comp
-L CP C?
+L CP C5
 U 1 1 5568F47F
 P 4800 3900
-F 0 "C?" H 4825 4000 50  0000 L CNN
+F 0 "C5" H 4825 4000 50  0000 L CNN
 F 1 "250u" H 4825 3800 50  0000 L CNN
 F 2 "" H 4838 3750 30  0000 C CNN
@@
 	4800 3750 4800 3700
 $Comp
-L +12V #PWR?
+L +12V #PWR21
 U 1 1 5568F497
 P 4800 2825
-F 0 "#PWR?" H 4800 2675 50  0001 C CNN
+F 0 "#PWR21" H 4800 2675 50  0001 C CNN
 F 1 "+12V" H 4800 2965 50  0000 C CNN
 F 2 "" H 4800 2825 60  0000 C CNN
@@
 $EndComp
 $Comp
-L GND #PWR?
+L GND #PWR23
 U 1 1 5568F49D
 P 5375 3250
-F 0 "#PWR?" H 5375 3000 50  0001 C CNN
+F 0 "#PWR23" H 5375 3000 50  0001 C CNN
 F 1 "GND" H 5375 3100 50  0000 C CNN
 F 2 "" H 5375 3250 60  0000 C CNN
@@
 $EndComp
 $Comp
-L CP C?
+L CP C4
 U 1 1 5568F4A3
 P 4800 3025
-F 0 "C?" H 4825 3125 50  0000 L CNN
+F 0 "C4" H 4825 3125 50  0000 L CNN
 F 1 "250u" H 4825 2925 50  0000 L CNN
 F 2 "" H 4838 2875 30  0000 C CNN
@@
 $EndComp
 $Comp
-L CONN_01X02 P?
+L CONN_01X02 P3
 U 1 1 5568F4AA
 P 4150 2975
-F 0 "P?" H 4150 3125 50  0000 C CNN
+F 0 "P3" H 4150 3125 50  0000 C CNN
 F 1 "CONN_01X02" V 4250 2975 50  0000 C CNN
 F 2 "" H 4150 2975 60  0000 C CNN
@@
 	4350 3175 5375 3175
 Wire Wire Line
-	4350 2875 4350 2925
+	4350 2425 4350 2925
 Connection ~ 4800 2875
 Wire Wire Line
@@
 Connection ~ 4800 3175
 $Comp
-L LM7810CT U?
+L LM7810CT U3
 U 1 1 5568F4BB
 P 5375 2925
-F 0 "U?" H 5175 3125 40  0000 C CNN
+F 0 "U3" H 5175 3125 40  0000 C CNN
 F 1 "LM7810CT" H 5375 3125 40  0000 L CNN
 F 2 "TO-220" H 5375 3025 30  0000 C CIN
@@
 $EndComp
 $Comp
-L +10 #PWR?
+L +10 #PWR25
 U 1 1 5568F4C2
 P 5950 2825
-F 0 "#PWR?" H 5950 2675 50  0001 C CNN
+F 0 "#PWR25" H 5950 2675 50  0001 C CNN
 F 1 "+10" H 5950 2975 50  0000 C CNN
 F 2 "" H 5950 2825 60  0000 C CNN
@@
 Text Notes 2875 3025 0    60   Italic 12
 Main Power Connector
+$Comp
+L LED D?
+U 1 1 55AC1458
+P 4675 2075
+F 0 "D?" H 4675 2175 50  0000 C CNN
+F 1 "LED" H 4675 1975 50  0000 C CNN
+F 2 "" H 4675 2075 60  0000 C CNN
+F 3 "" H 4675 2075 60  0000 C CNN
+	1    4675 2075
+	-1   0    0    1
+$EndComp
+$Comp
+L R_Small R?
+U 1 1 55AC1493
+P 4350 2325
+F 0 "R?" H 4380 2345 50  0000 L CNN
+F 1 "R_Small" H 4380 2285 50  0000 L CNN
+F 2 "" H 4350 2325 60  0000 C CNN
+F 3 "" H 4350 2325 60  0000 C CNN
+	1    4350 2325
+	1    0    0    -1
+$EndComp
+Connection ~ 4350 2875
+Wire Wire Line
+	4350 2225 4350 2075
+Wire Wire Line
+	4350 2075 4475 2075
+Wire Wire Line
+	4875 2075 5050 2075
+Wire Wire Line
+	5050 2075 5050 3175
+Connection ~ 5050 3175
 $EndSCHEMATC
